File: schematic/matrix_clock_kicad/matrix_clock_kicad.kicad_sch (KiCad schematic)
At the start: 7 parts, among them J1 LED Connector, J2 RTC, SW1 SELECT, SW2 SELECT, SW3 RESET, U1 Pico

Commit message: Completed PCB layout
Parts:
- U1: footprint PI Pico:RPi_Pico_SMD_TH -> Raspberry_Pi_Pico:RPi_Pico_SMD_TH
Changed lines of the file:
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@@
     (property "Reference" "U1" (id 0) (at 110.49 69.85 0))
     (property "Value" "Pico" (id 1) (at 110.49 72.39 0))
-    (property "Footprint" "PI Pico:RPi_Pico_SMD_TH" (id 2) (at 110.49 101.6 90)
+    (property "Footprint" "Raspberry_Pi_Pico:RPi_Pico_SMD_TH" (id 2) (at 110.49 101.6 90)
       (effects (font (size 1.27 1.27)) hide)
     )
@@
     )
     (path "/588e08bc-80dd-4d59-ac18-24f0d8657078"
-      (reference "U1") (unit 1) (value "Pico") (footprint "PI Pico:RPi_Pico_SMD_TH")
-    )
-  )
+      (reference "U1") (unit 1) (value "Pico") (footprint "Raspberry_Pi_Pico:RPi_Pico_SMD_TH")
+    )
+  )
