File: schematic/led_matrix_32x64_kicad/led_matrix_32x64_kicad.kicad_pcb (KiCad board)
At the start: 2 copper layers, 70.1 x 62 mm, 11 parts, among them J1 LED Interface, J2 RTC, J3 INTERFACE, J4 LEDPWR, SW3 RESET, U1 Pico, U2 NCP380

Commit message: update kicad schematin to tie MCP380 enable to ground
Parts:
- removed R1: 10k, Resistor_SMD:R_0805_2012Metric_Pad1.20x1.40mm_HandSolder
- C1: moved to F.Cu
- moved C1 0.21 mm to (115.3, 85.3)
Connections:
- U2 pad 4: /EN -> GND
Routing:
- net /EN: track 3.30 -> 0.00 mm
- net GND: track 332.3 -> 333.7 mm
